File: digikey_water-alarm.kicad_pcb (KiCad board)
At the start: 2 copper layers, 30 x 32.7 mm, 8 parts, among them J1 Jack-DC, J2 Screw_Terminal_01x02, Q1 2N7000

Commit message: done. gerber files included
Other:
- board text added: "vNOV 2025 Justin Kim"
